Commit message: Updates package name ransac_project to ransac_corridor_control. Added headless gazebo mode to lauch files. Fixed hokuyo sample/resolution bad value parameters...

File: src/vero_sim/urdf/hokuyo.urdf.xacro (robot description, xacro)
@@ -1,7 +1,6 @@
 <?xml version="1.0"?>
 <robot name="sensor_hokuyo" xmlns:xacro="http://www.ros.org/wiki/xacro">
- <!--  <xacro:include filename="$(find turtlebot_description)/urdf/turtlebot_gazebo.urdf.xacro"/>
-  <xacro:include filename="$(find turtlebot_description)/urdf/turtlebot_properties.urdf.xacro"/>
- -->
+  <!-- Import Rviz colors -->
+  <xacro:include filename="$(find vero_sim)/urdf/materials.xacro" />
   <!-- Hokuyo 2D LIDAR -->
   <xacro:macro name="sensor_hokuyo" params="name parent_link x y z roll pitch yaw">
@@ -14,7 +13,7 @@
       <visual>
         <geometry>
-          <box size="0.01 0.05 0.06" />
+          <box size="0.10 0.10 0.10" />
         </geometry>
-        <material name="Green" />
+        <material name="blue" />
       </visual>
       <inertial>
@@ -37,5 +36,5 @@
           <scan>
             <horizontal>
-              <samples>180</samples>
+              <samples>360</samples>
               <resolution>1</resolution>
               <min_angle>-1.570796</min_angle>
@@ -48,9 +47,9 @@
             <resolution>0.01</resolution>
           </range>
-<!--           <noise>
-            <type>Gaussian</type>
-            <mean>0.0</mean>
-            <stddev>0.01</stddev>
-          </noise> -->
+          <!--<noise>-->
+            <!--<type>Gaussian</type>-->
+            <!--<mean>0.0</mean>-->
+            <!--<stddev>0.01</stddev>-->
+          <!--</noise> -->
         </ray>
         <!--<plugin name="${name}_hokuyo_node" filename="libgazebo_ros_gpu_laser.so">-->

File: src/vero_sim/urdf/vero.urdf.xacro (robot description, xacro)
@@ -2,12 +2,11 @@
 <robot name="mkz" xmlns:xacro="http://www.ros.org/wiki/xacro" >
   <!-- Necessary includes -->
-  <xacro:arg name="urdf_model" default="$(find vero_sim)/urdf/mkz.urdf.xacro"/>
   <xacro:include filename="$(find dbw_mkz_description)/urdf/vehicle_structure.urdf.xacro" />
   <xacro:include filename="$(find dbw_mkz_description)/urdf/vehicle_gazebo.urdf.xacro" />
   <!-- Bolt-on sensors go here -->
-  <xacro:include filename="$(find dbw_mkz_description)/urdf/vehicle_sensors.urdf.xacro" />
+  <!--<xacro:include filename="$(find dbw_mkz_description)/urdf/vehicle_sensors.urdf.xacro" />-->
   <xacro:include filename="$(find vero_sim)/urdf/hokuyo.urdf.xacro" />
-  <xacro:dbw_mkz_camera name="front_camera" parent_link="base_footprint" x="2.0" y="0" z="1.3" roll="0" pitch="0.6" yaw="0" />
-  <xacro:dbw_mkz_gps name="perfect_gps" parent_link="base_footprint" x="0.6" y="0" z="1.45" rate="50.0" ref_lat="45.0" ref_lon="-81.0" />
-  <xacro:sensor_hokuyo name="hokuyo" parent_link="base_footprint" x="4.0" y="0.0" z="0.6" roll="0" pitch="0.0" yaw="0" />
+  <!--<xacro:dbw_mkz_camera name="front_camera" parent_link="base_footprint" x="2.0" y="0" z="1.3" roll="0" pitch="0.6" yaw="0" />-->
+  <!--<xacro:dbw_mkz_gps name="perfect_gps" parent_link="base_footprint" x="0.6" y="0" z="1.45" rate="50.0" ref_lat="45.0" ref_lon="-81.0" />-->
+  <xacro:sensor_hokuyo name="hokuyo" parent_link="base_footprint" x="3.86" y="0.0" z="0.6" roll="0.0" pitch="0.0" yaw="0.0" />
 </robot>
